File: KiCad/_autosave-PVDX Compute Board.kicad_pcb (KiCad board)
At the start: 2 copper layers, 66.5 x 64 mm, 47 parts, among them IC1 MIC5350-SGYMT-TR, J1 Conn_02x06_Counter_Clockwise, J2 USB_C_Receptacle_USB2.0_14P, J3 Conn_01x07, J4 Conn_01x06, J5 Conn_02x08_Odd_Even, J6 Conn_02x11_Counter_Clockwise, U1 EM008LX, U2 EM008LX, U3 EM008LX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

Commit message: update draft to 11/13 version
Parts:
- removed J5: Conn_02x08_Odd_Even, Connector_Harwin:Harwin_Gecko-G125-FVX1605L0X_2x08_P1.25mm_Vertical
- added C5: 0.1 uF, Capacitor_SMD:C_0201_0603Metric, F.Cu at (148.3, 54.5)
- added C6: 0.1 uF, Capacitor_SMD:C_0201_0603Metric, F.Cu at (152.8, 54.5)
- added C7: 0.1 uF, Capacitor_SMD:C_0201_0603Metric, F.Cu at (148.3, 75.0)
- added C8: 0.1 uF, Capacitor_SMD:C_0201_0603Metric, F.Cu at (154.8, 75.0)
- added R16: 10K, Resistor_SMD:R_0603_1608Metric, F.Cu at (151.8, 63.0)
- added R17: 10K, Resistor_SMD:R_0603_1608Metric, F.Cu at (151.7, 74.5)
- added U5: TXS0108EPW, Package_SO:TSSOP-20_4.4x6.5mm_P0.65mm, F.Cu at (151.5, 58.5)
- added U6: TXS0108EPW, Package_SO:TSSOP-20_4.4x6.5mm_P0.65mm, F.Cu at (151.5, 70.0)
- added U7: TMUX1108PW, Package_SO:TSSOP-16_4.4x5mm_P0.65mm, F.Cu at (205.1, 92.0)
- moved CIN1 61.9 mm to (216.8, 58.5)
- moved CIN2 61.9 mm to (216.8, 60.3)
- moved J1 61.9 mm to (213.8, 59.1)
- moved R7 61.9 mm to (213.4, 68.8)
- moved J6 45.1 mm to (173.0, 93.0), turned to 180 degrees
- moved J3 29.3 mm to (152.9, 44.0), turned to 90 degrees
- moved H3 22.5 mm to (216.1, 96.6)
- moved H4 17.0 mm to (144.4, 96.5)
- moved H2 14.7 mm to (216.1, 24.9)
- moved R3 10.7 mm to (158.0, 48.0), turned to 0 degrees
- moved R8 4.10 mm to (166.0, 29.5), turned to -90 degrees
- moved R14 3.41 mm to (202.0, 72.5), turned to -90 degrees
- moved J4 2.71 mm to (185.3, 25.2)
- moved H1 2.36 mm to (144.4, 24.9)
- moved R2 2.00 mm to (165.5, 63.0)
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Connections:
- J6 pad 1: unconnected-(J6-Pin_1-Pad1) -> PHOTO01A
- J6 pad 10: unconnected-(J6-Pin_10-Pad10) -> PHOTO10A
- J6 pad 11: unconnected-(J6-Pin_11-Pad11) -> PHOTO11A
- J6 pad 12: unconnected-(J6-Pin_12-Pad12) -> PHOTO11B
- J6 pad 13: unconnected-(J6-Pin_13-Pad13) -> PHOTO10B
- J6 pad 14: unconnected-(J6-Pin_14-Pad14) -> PHOTO09B
- J6 pad 15: unconnected-(J6-Pin_15-Pad15) -> PHOTO08B
- J6 pad 16: unconnected-(J6-Pin_16-Pad16) -> PHOTO07B
- J6 pad 17: unconnected-(J6-Pin_17-Pad17) -> PHOTO06B
- J6 pad 18: unconnected-(J6-Pin_18-Pad18) -> PHOTO05B
- J6 pad 19: unconnected-(J6-Pin_19-Pad19) -> PHOTO04B
- J6 pad 2: unconnected-(J6-Pin_2-Pad2) -> PHOTO02A
- J6 pad 20: unconnected-(J6-Pin_20-Pad20) -> PHOTO03B
- J6 pad 21: unconnected-(J6-Pin_21-Pad21) -> PHOTO02B
- J6 pad 22: unconnected-(J6-Pin_22-Pad22) -> PHOTO01B
- J6 pad 3: unconnected-(J6-Pin_3-Pad3) -> PHOTO03A
- J6 pad 4: unconnected-(J6-Pin_4-Pad4) -> PHOTO04A
- J6 pad 5: unconnected-(J6-Pin_5-Pad5) -> PHOTO05A
- J6 pad 6: unconnected-(J6-Pin_6-Pad6) -> PHOTO06A
- J6 pad 7: unconnected-(J6-Pin_7-Pad7) -> PHOTO07A
- J6 pad 8: unconnected-(J6-Pin_8-Pad8) -> PHOTO08A
- J6 pad 9: unconnected-(J6-Pin_9-Pad9) -> PHOTO09A
- R1 pad 2: PC14 -> PC14 1V8
- R2 pad 2: PC15 -> PC15 1V8
- R3 pad 2: PC12 -> PC12 1V8
- R4 pad 1: 1V8 -> PC05 1V8
- R4 pad 2: PC05 -> 1V8
- R5 pad 1: 1V8 -> PC07 1V8
- R5 pad 2: PC07 -> 1V8
- R6 pad 1: 1V8 -> PC10 1V8
- R6 pad 2: PC10 -> 1V8
- U1 pad 1: PC04 -> PC04 1V8
- U1 pad 2: PD11 (MISO) -> PD11 (MISO) 1V8
- U1 pad 3: PC14 -> PC14 1V8
- U1 pad 5: PD08 (MOSI) -> PD08 (MOSI) 1V8
- U1 pad 6: PD09 (SCK) -> PD09 (SCK) 1V8
- U1 pad 7: PC05 -> PC05 1V8
- U2 pad 1: PC06 -> PC06 1V8
- U2 pad 2: PD11 (MISO) -> PD11 (MISO) 1V8
- U2 pad 3: PC15 -> PC15 1V8
- U2 pad 5: PD08 (MOSI) -> PD08 (MOSI) 1V8
- U2 pad 6: PD09 (SCK) -> PD09 (SCK) 1V8
- U2 pad 7: PC07 -> PC07 1V8
- U3 pad 1: PC11 -> PC11 1V8
- U3 pad 2: PD11 (MISO) -> PD11 (MISO) 1V8
- U3 pad 3: PC12 -> PC12 1V8
- U3 pad 5: PD08 (MOSI) -> PD08 (MOSI) 1V8
- U3 pad 6: PD09 (SCK) -> PD09 (SCK) 1V8
- U3 pad 7: PC10 -> PC10 1V8
Routing:
- net GND: track 292.5 -> 370.3 mm, vias 30 -> 25
- net 5V: track 48.3 -> 123.1 mm, vias 3 -> 6
- net PD21: track 82.2 -> 15.8 mm
- net PD09 (SCK) 1V8: track 0.00 -> 56.8 mm, vias 0 -> 4
- net PC05 1V8: track 0.00 -> 56.5 mm, vias 0 -> 2
- net PD08 (MOSI) 1V8: track 0.00 -> 55.7 mm, vias 0 -> 5
- net 1V8: track 71.7 -> 118.9 mm, vias 2 -> 6
- net PA16 (SCL): track 63.4 -> 17.3 mm, vias 2 -> 0
- net PD11 (MISO) 1V8: track 0.00 -> 44.1 mm, vias 0 -> 5
- net PA17 (SDA): track 62.8 -> 20.6 mm, vias 2 -> 0
- net AIN00: track 0.00 -> 40.5 mm
- net PC05: track 16.9 -> 52.5 mm, vias 2 -> 0
- net PC12 1V8: track 0.00 -> 35.1 mm, vias 0 -> 2
- net 3V3: track 233.4 -> 267.6 mm, vias 9 -> 13
- net PC10 1V8: track 0.00 -> 31.0 mm, vias 0 -> 2
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Other:
- board size 66.5 x 64 mm -> 82.5 x 82.5 mm
- board text added: "3V3"
- board text added: "5V"
- board text added: "ARDUCAM"
- board text added: "CS"
- board text added: "DRDY"
- board text added: "GND"
- board text added: "MAGNETOMETER"
- board text added: "MISO"
- board text added: "MOSI"
- board text added: "OLED"
- board text added: "P01A"
- board text added: "P01B"
- board text added: "P02A"
- board text added: "P02B"
- board text added: "P03A"
- board text added: "P03B"
- board text added: "P04A"
- board text added: "P04B"
- board text added: "P05A"
- board text added: "P05B"
- board text added: "P06A"
- board text added: "P06B"
- board text added: "P07A"
- board text added: "P07B"
- board text added: "P08A"
- board text added: "P08B"
- board text added: "P09A"
- board text added: "P09B"
- board text added: "P10A"
- board text added: "P10B"
- board text added: "P11A"
- board text added: "P11B"
- board text added: "PHOTODIODES"
- board text added: "REXT"
- board text added: "SCK"
- board text added: "SCL"
- board text added: "SDA"
- board text added: "~{CS}"
- board text added: "~{D/C}"
- board text added: "~{RES}"
