File: SAMD51_dev_board/peripherals.kicad_sch (KiCad schematic)
At the start: 23 parts, among them IC1 MCP1603-330I_MC, IC2 MCP1603-180I_MC, J1 Conn_02x08_Top_Bottom, J2 USB4105-GF-A, J3 FTSH-105-01-L-DV-007-K

Commit message: Update LED resistor values
Parts:
- R1, R2, R3, R4: value 1K -> 330
Other:
- note added: "1.85V"
- note added: "1.9V"
- note added: "2V"
Changed lines of the file:
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@@
 		)
 	)
+	(text "1.85V\n"
+		(exclude_from_sim no)
+		(at 96.774 175.26 0)
+		(effects
+			(font
+				(size 1.27 1.27)
+			)
+		)
+	)
 	(text "J LINK / SWD"
 		(exclude_from_sim no)
@@
 		)
 	)
+	(text "1.9V\n"
+		(exclude_from_sim no)
+		(at 64.262 174.752 0)
+		(effects
+			(font
+				(size 1.27 1.27)
+			)
+		)
+	)
 	(text "PVDX COMPUTE BOARD\n"
 		(exclude_from_sim no)
@@
 		)
 	)
+	(text "1.85V\n"
+		(exclude_from_sim no)
+		(at 95.758 195.072 0)
+		(effects
+			(font
+				(size 1.27 1.27)
+			)
+		)
+	)
 	(text "Milan Capoor"
 		(exclude_from_sim no)
@@
 		)
 	)
+	(text "2V\n"
+		(exclude_from_sim no)
+		(at 52.832 194.564 0)
+		(effects
+			(font
+				(size 1.27 1.27)
+			)
+		)
+	)
 	(junction
 		(at 276.86 74.93)
@@
 			)
 		)
-		(property "Value" "1K"
+		(property "Value" "330"
 			(at 89.916 179.07 90)
 			(show_name no)
@@
 			)
 		)
-		(property "Value" "1K"
+		(property "Value" "330"
 			(at 57.15 179.324 90)
 			(show_name no)
@@
 		)
 		(property "Value" "ORANGE"
-			(at 100.076 194.818 0)
+			(at 108.966 196.342 0)
 			(show_name no)
 			(do_not_autoplace no)
@@
 			)
 		)
-		(property "Value" "1K"
+		(property "Value" "330"
 			(at 90.17 190.5 90)
 			(show_name no)
@@
 			)
 		)
-		(property "Value" "1K"
+		(property "Value" "330"
 			(at 53.594 189.23 90)
 			(show_name no)
