File: Compute Board/peripherals.kicad_sch (KiCad schematic)
At the start: 61 parts, among them IC1 MCP1603-330I_MC, IC2 MCP1603-180I_MC, J1 USB_C_Receptacle_USB2.0_14P, J2 FTSH-105-01-L-DV-007-K, U1 EM008LX, U10 Sen-Z-f, U2 EM008LX, U3 EM008LX, U4 TXS0108EPW, U5 TXS0108EPW, U6 SCH16T-K01-1, U7 MagI2C, U8 Sen-XY-f, U9 Sen-XY-f

Commit message: Push layout-ready schematics and partial routing
Parts:
- removed C13, C17: 4.7 uF, Capacitor_SMD:C_0402_1005Metric, symbol Device:C
- removed IC1: MCP1603-330I_MC, MPC1603:MPC1603-330, symbol MCP1603:MCP1603-330I_MC
- removed J1: USB_C_Receptacle_USB2.0_14P, Connector_USB:USB_C_Receptacle_HCTL_HC-TYPE-C-16P-01A, symbol Connector:USB_C_Receptacle_USB2.0_14P
- removed L1: 4.7 uH, Inductor_SMD:L_0402_1005Metric, symbol Device:L
- removed R10, R9: 5.1K, Resistor_SMD:R_0402_1005Metric, symbol Device:R
- removed R11, R12: 22, Resistor_SMD:R_0402_1005Metric, symbol Device:R
- added J12: Conn_01x03, Connector_PinSocket_2.54mm:PinSocket_1x03_P2.54mm_Vertical, symbol Connector_Generic:Conn_01x03
- C1, C10, C11, C12, C14, C15, C16, C18, C2, C3, C4, C5, C6, C7, C8, C9: footprint Capacitor_SMD:C_0402_1005Metric -> Capacitor_SMD:C_0603_1608Metric
- D1, D2, D3, D4: footprint LED_SMD:LED_0402_1005Metric -> LED_SMD:LED_0603_1608Metric
- H1, H2, H3, H4: footprint MountingHole:MountingHole_2.1mm -> MountingHole:MountingHole_3.2mm_M3
- L2: footprint Inductor_SMD:L_0402_1005Metric -> Inductor_SMD:L_0603_1608Metric
- R1, R13, R14, R15, R16, R17, R18, R19, R2, R3, R4, R5, R6, R7, R8: footprint Resistor_SMD:R_0402_1005Metric -> Resistor_SMD:R_0603_1608Metric
Connections:
- net +3V3: now also C14.1, IC2.2 (NC_1), J12.1 (Pin_1)
- net +5V: now also J12.3 (Pin_3); no longer C14.1, IC2.2 (NC_1)
- net GND: now also J12.2 (Pin_2)
- net at R16.2, U7.11 (YNP), U9.1: no longer R17.2, U7.12 (YNN), U9.2
- net GYRO DRDY renamed GYRO ~{DRDY}
- net LED ORANGE 1 renamed LED ~{ORANGE 1}
- net LED ORANGE 2 renamed LED ~{ORANGE 2}
- net LED RED renamed LED ~{RED}
- net MAG DRDY renamed MAG ~{DRDY}
- new net: R17.2, U7.12 (YNN), U9.2
- no-connect marks 20 -> 17
Other:
- note added: "ACCELEROMETER"
- note added: "POWER AND REGULATORS"
- note added: "TODO: confirm LED schematic"
- note removed: "GYRSOSCOPE"
- note removed: "TODO: change power connection to match structures' spec for board power. Deicde if you want to generate 5V, 3V3, and 1V8 on PDB or in-situ"
- note removed: "TODO: check with FSW if these should be pullup/down and adjust schematic accordingly"
- note removed: "TODO: confirm mounting hole size with structures (these are 2.1mm)"
- note removed: "TODO: review the SAMD51 dev board schematic in commit c98bf0a to adjust USB-C and regulators (if using)"
- note removed: "TODO: these don't have pins allocated on the samd51 and were added for forwards-compatibility; check if FSW actually wants them / decide what to do with them"
- note removed: "USB CONNECTION AND REGULATORS"
- moved on the sheet: C14, C18
